Commit message: ..

File: install/igus_rebel_description/share/igus_rebel_description/urdf/igus_rebel2.urdf (robot description, URDF)
Before this commit: robot igus_rebel, 12 links, 11 joints
Links:
- link base_link: geometry collision cylinder length=0.1 radius=0.09; visual mesh filename=file://$(find igus_rebel_description)/meshes/robolink_rebel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
- link link1: geometry collision box size=0.1 0.03 0.1; visual mesh filename=file://$(find igus_rebel_description)/meshes/robolink_rebel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
- link link2: geometry collision cylinder length=0.18 radius=0.06; visual mesh filename=file://$(find igus_rebel_description)/meshes/robolink_rebel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
- link link3: geometry collision box size=0.1 0.03 0.1; visual mesh filename=file://$(find igus_rebel_description)/meshes/robolink_rebel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
- link link4: geometry collision cylinder length=0.1 radius=0.05; visual mesh filename=file://$(find igus_rebel_description)/meshes/robolink_rebel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
- link link5: geometry collision box size=0.1 0.03 0.1; visual mesh filename=file://$(find igus_rebel_description)/meshes/robolink_rebel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
- link link6: geometry collision cylinder length=0.065 radius=0.04; visual mesh filename=file://$(find igus_rebel_description)/meshes/robolink_rebel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
- link motor1: geometry collision cylinder length=0.065 radius=0.05; visual mesh filename=file://$(find igus_rebel_description)/meshes/robolink_rebel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
- link motor2: geometry collision cylinder length=0.065 radius=0.05; visual mesh filename=file://$(find igus_rebel_description)/meshes/robolink_rebel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
- link motor3: geometry collision cylinder length=0.065 radius=0.05; visual mesh filename=file://$(find igus_rebel_description)/meshes/robolink_rebel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
- link motor4: geometry collision cylinder length=0.065 radius=0.05; visual mesh filename=file://$(find igus_rebel_description)/meshes/robolink_rebel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
- link motor5: geometry collision cylinder length=0.065 radius=0.04; visual mesh filename=file://$(find igus_rebel_description)/meshes/robolink_rebel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
Joints:
- joint joint1: axis 0 0 -1 -> 0 0 1
